File: sp6641b.sch (EAGLE design)
At the start: 11 parts

Commit message: Modified board layouts
Parts:
- removed GND, GND_IN, VBATT, VOUT: WIREPAD2,54/1,0, wirepad:WIREPAD2,54/1,0
- added J1, J2: (no value), SparkFun-Connectors:M02PTH
- U$1: value SP6641A -> SP6641B
Connections:
- net GND: now also J1.2, J2.2; no longer GND.P, GND_IN.P
- net VBATT: now also J1.1; no longer VBATT.P
- net VOUT: now also J2.1; no longer VOUT.P
Changed lines of the file:
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@@
 <layer number="56" name="wert" color="7" fill="1" visible="no" active="no"/>
 <layer number="57" name="tCAD" color="7" fill="1" visible="no" active="no"/>
+<layer number="59" name="tCarbon" color="7" fill="1" visible="no" active="no"/>
+<layer number="60" name="bCarbon" color="7" fill="1" visible="no" active="no"/>
+<layer number="90" name="Modules" color="5" fill="1" visible="yes" active="yes"/>
 <layer number="91" name="Nets" color="2" fill="1" visible="yes" active="yes"/>
 <layer number="92" name="Busses" color="1" fill="1" visible="yes" active="yes"/>
@@
 <layer number="112" name="tSilk" color="7" fill="1" visible="yes" active="yes"/>
 <layer number="113" name="IDFDebug" color="4" fill="1" visible="yes" active="yes"/>
+<layer number="114" name="Badge_Outline" color="7" fill="1" visible="yes" active="yes"/>
+<layer number="115" name="ReferenceISLANDS" color="7" fill="1" visible="yes" active="yes"/>
 <layer number="116" name="Patch_BOT" color="9" fill="4" visible="yes" active="yes"/>
+<layer number="118" name="Rect_Pads" color="7" fill="1" visible="yes" active="yes"/>
 <layer number="121" name="_tsilk" color="7" fill="1" visible="yes" active="yes"/>
 <layer number="122" name="_bsilk" color="7" fill="1" visible="yes" active="yes"/>
@@
 <layer number="127" name="_tValues" color="7" fill="1" visible="yes" active="yes"/>
 <layer number="128" name="_bValues" color="7" fill="1" visible="yes" active="yes"/>
+<layer number="129" name="Mask" color="7" fill="1" visible="yes" active="yes"/>
 <layer number="131" name="tAdjust" color="7" fill="1" visible="yes" active="yes"/>
 <layer number="132" name="bAdjust" color="7" fill="1" visible="yes" active="yes"/>
@@
 <layer number="251" name="SMDround" color="12" fill="11" visible="no" active="no"/>
 <layer number="254" name="cooling" color="7" fill="1" visible="yes" active="yes"/>
+<layer number="255" name="routoute" color="7" fill="1" visible="yes" active="yes"/>
 </layers>
 <schematic xreflabel="%F%N/%S.%C%R" xrefpart="/%S.%C%R">
@@
 </classes>
 <parts>
-<part name="U$1" library="Sipex Custom" deviceset="SP6641" device="SP6641A/B" value="SP6641A"/>
+<part name="U$1" library="Sipex Custom" deviceset="SP6641" device="SP6641A/B" value="SP6641B"/>
 <part name="C1" library="SparkFun" deviceset="CAP" device="0805" value="100uF"/>
 <part name="C2" library="SparkFun" deviceset="CAP" device="0805" value="100uF"/>
@@
 <part name="V_BATT_IN" library="SparkFun" deviceset="3.3V" device="" value="1.5v-3.0v"/>
 <part name="GND3" library="SparkFun" deviceset="GND" device=""/>
-<part name="VOUT" library="wirepad" deviceset="WIREPAD" device="2,54/1,0" value=""/>
-<part name="GND_IN" library="wirepad" deviceset="WIREPAD" device="2,54/1,0" value=""/>
-<part name="VBATT" library="wirepad" deviceset="WIREPAD" device="2,54/1,0" value=""/>
-<part name="GND" library="wirepad" deviceset="WIREPAD" device="2,54/1,0" value=""/>
 <part name="D1" library="diode" deviceset="MBR0520LT" device="" value="MBR0520"/>
 <part name="R1" library="SparkFun-Resistors" deviceset="0.3OHM-1/8W-1%(0805)" device="" value="10"/>
 <part name="C3" library="SparkFun" deviceset="CAP" device="0805" value="1uF"/>
 <part name="GND4" library="SparkFun" deviceset="GND" device=""/>
+<part name="J1" library="SparkFun-Connectors" deviceset="M02" device="PTH"/>
+<part name="J2" library="SparkFun-Connectors" deviceset="M02" device="PTH"/>
 </parts>
 <sheets>
@@
 <instance part="V_BATT_IN" gate="G$1" x="83.82" y="36.83"/>
 <instance part="GND3" gate="1" x="19.05" y="-12.7"/>
-<instance part="VOUT" gate="G$1" x="110.49" y="15.24" rot="R180"/>
-<instance part="GND_IN" gate="G$1" x="110.49" y="34.29" rot="R180"/>
-<instance part="VBATT" gate="G$1" x="110.49" y="40.64" rot="R180"/>
-<instance part="GND" gate="G$1" x="110.49" y="8.89" rot="R180"/>
 <instance part="D1" gate="G$1" x="7.62" y="25.4" rot="R270"/>
 <instance part="R1" gate="G$1" x="19.05" y="15.24" rot="R90"/>
 <instance part="C3" gate="G$1" x="29.21" y="17.78" rot="R180"/>
 <instance part="GND4" gate="1" x="29.21" y="7.62"/>
+<instance part="J1" gate="G$1" x="67.31" y="1.27" rot="R180"/>
+<instance part="J2" gate="G$1" x="67.31" y="-13.97" rot="R180"/>
 </instances>
 <busses>
@@
 </segment>
 <segment>
-<pinref part="GND_IN" gate="G$1" pin="P"/>
-<wire x1="107.95" y1="34.29" x2="101.6" y2="34.29" width="0.1524" layer="91"/>
-<junction x="101.6" y="34.29"/>
+<wire x1="59.69" y1="-1.27" x2="53.34" y2="-1.27" width="0.1524" layer="91"/>
+<junction x="53.34" y="-1.27"/>
+<pinref part="J1" gate="G$1" pin="2"/>
 </segment>
 <segment>
@@
 </segment>
 <segment>
-<pinref part="GND" gate="G$1" pin="P"/>
-<wire x1="107.95" y1="8.89" x2="101.6" y2="8.89" width="0.1524" layer="91"/>
-<junction x="101.6" y="8.89"/>
+<wire x1="59.69" y1="-16.51" x2="53.34" y2="-16.51" width="0.1524" layer="91"/>
+<junction x="53.34" y="-16.51"/>
+<pinref part="J2" gate="G$1" pin="2"/>
 </segment>
 </net>
@@
 </segment>
 <segment>
-<pinref part="VBATT" gate="G$1" pin="P"/>
-<wire x1="107.95" y1="40.64" x2="101.6" y2="40.64" width="0.1524" layer="91"/>
-<junction x="101.6" y="40.64"/>
+<wire x1="59.69" y1="1.27" x2="53.34" y2="1.27" width="0.1524" layer="91"/>
+<junction x="53.34" y="1.27"/>
+<pinref part="J1" gate="G$1" pin="1"/>
 </segment>
 </net>
@@
 <net name="VOUT" class="0">
 <segment>
-<pinref part="VOUT" gate="G$1" pin="P"/>
-<wire x1="107.95" y1="15.24" x2="101.6" y2="15.24" width="0.1524" layer="91"/>
-<junction x="101.6" y="15.24"/>
-</segment>
-<segment>
+<wire x1="59.69" y1="-13.97" x2="53.34" y2="-13.97" width="0.1524" layer="91"/>
+<junction x="53.34" y="-13.97"/>
+<pinref part="J2" gate="G$1" pin="1"/>
+</segment>
+<segment>
