File: lmr14206.sch (EAGLE design)
At the start: 12 parts

Commit message: Breakout board updates
Parts:
- added C6: 1uF, SparkFun-Capacitors:1UF-25V-10%(0805)"
- added D2: YELLOW, SparkFun-LED:LED-YELLOW1206
- added J3: (no value), SparkFun-Connectors:M02PTH
- added R3: 270k, SparkFun-Resistors:0.75OHM-1/4W-1%(0805)
- added R4: 680, SparkFun-Resistors:0.3OHM-1/8W-1%(0805)
- added R5: 34k, SparkFun-Resistors:0.75OHM-1/4W-1%(0805)
- C5: device SparkFun-Capacitors:10UF50V20%(1210) -> SparkFun-Capacitors:1UF-25V-10%(0805)"
- D1: value BAT20J -> (none); device SparkFun-DiscreteSemi:DIODE-SCHOTTKY-BAT20J -> SparkFun-DiscreteSemi:DIODESMB
Connections:
- removed net 5V: C3.1, C5.1, J2.1, L1.2, R1.2
- new net FB: R1.1, R2.2, R5.1, U$1.FB
- new net N$2: D2.A, R4.1
- new net N$5: C6.1, R3.1, U$1./SHDN
- new net VCC: C3.1, C5.1, J2.1, J3.1, L1.2, R1.2, R4.2
- net GND: now also C6.2, D2.C
- net N$1: now also J3.2, R5.2; no longer R1.1, R2.2, U$1.FB
- net VIN: now also R3.2; no longer U$1./SHDN
Other:
- note added: "* C2, C3, and C4 are X7R, low ESR ceramics * Place C2 close to the converter IC * R3/C6 form the soft start circuit, where 0.0v - 2.3v across C6 controls the start time"
- note added: "R1=R2((V OUT /0.765V)-1) R1 ~= 27k for 5.0V R1 ~= 15k for 3.3V"
- note removed: "* C2, C3, and C4 are X7R, low ESR ceramics"
- note removed: "R1=R2((V OUT /0.765V)-1)"
- note removed: "Vout ~= 5.15v"
- moved on the sheet: C2, C5, R1, R2
