File: xc9141-xc9142.sch (EAGLE design)
At the start: 7 parts

Commit message: Breakout board updates
Parts:
- added D1: YELLOW, SparkFun-LED:LED-YELLOW1206
- added R1: 680, SparkFun-Resistors:0.3OHM-1/8W-1%(0805)
Connections:
- new net N$1: D1.A, R1.1
- net 5V: now also R1.2
- net GND: now also D1.C
Changed lines of the file:
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@@
 <part name="SUPPLY3" library="SparkFun-Aesthetics" deviceset="V_BATT" device=""/>
 <part name="GND3" library="SparkFun-Aesthetics" deviceset="GND" device=""/>
+<part name="D1" library="SparkFun-LED" deviceset="LED-YELLOW" device="1206" value="YELLOW"/>
+<part name="R1" library="SparkFun-Resistors" deviceset="0.3OHM-1/8W-1%(0805)" device="" value="680"/>
+<part name="SUPPLY4" library="SparkFun-Aesthetics" deviceset="5V" device=""/>
+<part name="GND4" library="SparkFun-Aesthetics" deviceset="GND" device=""/>
 </parts>
 <sheets>
@@
 <instance part="SUPPLY3" gate="G$1" x="96.52" y="83.82"/>
 <instance part="GND3" gate="1" x="96.52" y="66.04"/>
+<instance part="D1" gate="G$1" x="119.38" y="35.56"/>
+<instance part="R1" gate="G$1" x="119.38" y="45.72" rot="R90"/>
+<instance part="SUPPLY4" gate="G$1" x="119.38" y="53.34"/>
+<instance part="GND4" gate="1" x="119.38" y="25.4"/>
 </instances>
 <busses>
@@
 <pinref part="GND3" gate="1" pin="GND"/>
 </segment>
+<segment>
+<pinref part="D1" gate="G$1" pin="C"/>
+<wire x1="119.38" y1="30.48" x2="119.38" y2="27.94" width="0.1524" layer="91"/>
+<pinref part="GND4" gate="1" pin="GND"/>
+</segment>
 </net>
 <net name="N$4" class="0">
@@
 <junction x="81.28" y="53.34"/>
 </segment>
+<segment>
+<pinref part="R1" gate="G$1" pin="2"/>
+<wire x1="119.38" y1="50.8" x2="119.38" y2="53.34" width="0.1524" layer="91"/>
+<pinref part="SUPPLY4" gate="G$1" pin="5V"/>
+</segment>
 </net>
 <net name="V_BATT" class="0">
@@
 </segment>
 </net>
+<net name="N$1" class="0">
+<segment>
+<pinref part="R1" gate="G$1" pin="1"/>
+<pinref part="D1" gate="G$1" pin="A"/>
+<wire x1="119.38" y1="40.64" x2="119.38" y2="38.1" width="0.1524" layer="91"/>
+</segment>
+</net>
